File: Mcu_V1/Mcu_V1.kicad_pcb (KiCad board)
At the start: 2 copper layers, 47.8 x 31.5 mm, 29 parts, among them J1 Conn_01x04_Pin, J2 Conn_01x09_Pin, J3 Conn_01x04_Pin, J4 Conn_02x03_Odd_Even, U1 24LC1025, U2 DS1337S_, U3 24LC1025, U4 ATMEGA328P-AU, Y1 32.768 KHz, Y2 16MHz

Commit message: update
Parts:
- moved J2 8.46 mm to (144.8, 105.0)
- moved J1 7.86 mm to (180.8, 93.4)
- moved BT1 7.86 mm to (142.4, 86.8)
- moved C1 7.86 mm to (157.4, 80.2)
- moved C2 7.86 mm to (170.2, 95.4)
- moved C3 7.86 mm to (161.4, 80.2)
- moved C4 7.86 mm to (170.2, 99.4)
- moved C5 7.86 mm to (165.6, 80.2)
- moved D1 7.86 mm to (174.2, 80.4)
- moved D2 7.86 mm to (170.0, 80.4)
- moved H1 7.86 mm to (182.6, 80.0)
- moved H2 7.86 mm to (140.0, 80.0)
- moved H3 7.86 mm to (182.6, 106.2)
- moved H4 7.86 mm to (140.0, 106.2)
- moved J4 7.86 mm to (178.3, 84.5)
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Routing:
- net /Vcc: track 0.00 -> 122.0 mm, vias 0 -> 3
- net GND: track 0.00 -> 103.1 mm, vias 0 -> 8
- net /SCK: track 0.00 -> 98.9 mm, vias 0 -> 2
- net /SDA: track 0.00 -> 66.6 mm, vias 0 -> 5
- net Net-(BT1-+): track 0.00 -> 65.8 mm
- net /RX: track 0.00 -> 31.1 mm, vias 0 -> 1
- net /TX: track 0.00 -> 29.7 mm, vias 0 -> 1
- net /D3: track 0.00 -> 26.5 mm, vias 0 -> 2
- net /RESET: track 0.00 -> 26.2 mm, vias 0 -> 2
- net Net-(U4-PB7): track 0.00 -> 25.7 mm, vias 0 -> 2
- net /D2: track 0.00 -> 25.7 mm, vias 0 -> 1
- net /MOSI: track 0.00 -> 22.8 mm
- net /D4: track 0.00 -> 22.7 mm, vias 0 -> 1
- net Net-(U4-PB6): track 0.00 -> 22.2 mm
- net /MISO: track 0.00 -> 17.9 mm, vias 0 -> 1
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- added copper zone on B.Cu, net GND
Other:
- board size 47.8 x 31.5 mm -> 47.8 x 31.4 mm

Commit message: 4 layer done
Parts:
- moved R1 6.81 mm to (147.5, 100.8)
- moved R2 6.80 mm to (152.1, 100.8), turned to 180 degrees
- moved U2 3.01 mm to (150.1, 95.6)
- moved H1 1.61 mm to (182.8, 78.4)
- moved H2 1.60 mm to (140.0, 78.4)
- moved H3 1.41 mm to (182.8, 107.6)
- moved H4 1.40 mm to (140.0, 107.6)
- moved Y2 0.82 mm to (161.8, 98.0)
Routing:
- net /Vcc: track 122.0 -> 5.64 mm, vias 3 -> 0
- net GND: track 103.1 -> 15.9 mm, vias 8 -> 0
- net /SCK: track 98.9 -> 17.5 mm, vias 2 -> 0
- net Net-(BT1-+): track 65.8 -> 0.00 mm
- net /SDA: track 66.6 -> 16.5 mm, vias 5 -> 0
- net /RESET: track 26.2 -> 0.00 mm, vias 2 -> 0
- net Net-(U4-PB7): track 25.7 -> 0.00 mm, vias 2 -> 0
- net /D2: track 25.7 -> 0.00 mm, vias 1 -> 0
- net /MOSI: track 22.8 -> 0.00 mm
- net Net-(U4-PB6): track 22.2 -> 0.00 mm
- net /MISO: track 17.9 -> 0.00 mm, vias 1 -> 0
- net Net-(U4-AREF): track 14.0 -> 0.00 mm, vias 2 -> 0
- net /D8: track 12.3 -> 20.6 mm, vias 1 -> 0
- net /TX: track 29.7 -> 37.1 mm, vias 1 -> 0
- net Net-(D1-K): track 4.97 -> 0.00 mm
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- removed copper zone on B.Cu, net GND
Other:
- board size 47.8 x 31.4 mm -> 48.8 x 35.2 mm
- copper layers 2 -> 4
